Commit message: distance input control

File: src/robot_description/urdf/arm_fp.urdf (robot description, URDF)
Before this commit: robot Assem1, 10 links, 9 joints
Links:
- added link base_inertia, mass 0.11758
- link base_link: mass 0.11758 -> None
Joints:
- added joint base_to_base_inertia: type fixed, parent base_link, child base_inertia, origin xyz=0 0 0 rpy=0 0 0
