Commit message: materi urdf magang

File: src/robot_description/urdf/arm_magang.urdf (robot description, URDF)
Before this commit: robot arm, 6 links, 5 joints
Links:
- removed link hand
- link forearm: geometry collision cylinder length=0.3 radius=0.03; visual cylinder length=0.3 radius=0.03
- link torso: geometry collision cylinder length=0.12 radius=0.03; visual cylinder length=0.12 radius=0.03
- link upper_arm: geometry collision cylinder length=0.3 radius=0.03; visual cylinder length=0.3 radius=0.03
Joints:
- removed joint wrist
- joint elbow: origin xyz=0.0 0.1 0.35 rpy=0 0 0 -> xyz=0 -0.055 0.1 rpy=0 0 0
- joint hip: origin xyz=0 0 0.05 rpy=0 0 0 -> xyz=0 0 0.11 rpy=0 0 0
- joint shoulder: origin xyz=0.0 -0.1 0.45 rpy=0 1.5708 0 -> xyz=0.02 0.06 0.06 rpy=0 1.5708 0
